Commit message: second commit

File: xacro/depthCamera1.xacro (robot description, xacro)
@@ -2,10 +2,10 @@
 <robot xmlns:xacro="http://www.ros.org/wiki/xacro">
     <xacro:macro name="depthCamera" params="camID name *origin">
-        <joint name="camera_joint_${name}" type="fixed">
+        <joint name="camera_joint_face" type="fixed">
             <xacro:insert_block name="origin"/>
             <parent link="trunk"/>
-            <child link="camera_${name}"/>
+            <child link="camera_face"/>
         </joint>
-        <link name="camera_${name}">
+        <link name="camera_face">
             <collision>
             <origin xyz="0 0 0" rpy="0 0 0"/>
@@ -33,9 +33,9 @@
         <link name="camera_optical_${name}">
         </link>
-        <gazebo reference="camera_${name}">
+        <gazebo reference="camera_face">
             <!-- <material>Gazebo/Black</material> -->
-            <sensor name="camera_${name}_camera" type="depth">
+            <sensor name="camera_face_camera" type="depth">
                 <!-- <pose> 0 0 0 0 0 0 </pose> -->
-                <update_rate>100</update_rate><!-- was 16 -->
+                <update_rate>10</update_rate><!-- was 16 -->
                 <camera>
                     <horizontal_fov>2.094</horizontal_fov>
@@ -80,6 +80,6 @@
                 -->
                 <!-- WE REPLACE IT WITH A NORMAL DEPTH CAMERA PLUGIN FOR NOW -->
-                <plugin name="camera_${name}_controller" filename="libgazebo_ros_camera.so">
-                    <frame_name>camera_optical_${name}</frame_name>
+                <plugin name="camera_face_controller" filename="libgazebo_ros_camera.so">
+                    <frame_name>camera_optical_face</frame_name>
                     <min_depth>0.1</min_depth>
                     <max_depth>100</max_depth>

File: xacro/gazebo.xacro (robot description, xacro)
@@ -24,6 +24,8 @@
     <!-- ADDED START -->
         <!-- GAZEBO DIFF DRIVE -->
+        <!-- USING THIS AS A WORKAROUND UNTIL HIGH LEVEL CONTROL IS ESTABLISHED -->
     <gazebo>
         <plugin name='diff_drive' filename='libgazebo_ros_diff_drive.so'>
+            <updateRate>10</updateRate><!-- was 20 -->
             <!-- Wheel Information -->
             <left_joint>left_wheel_joint</left_joint>
@@ -36,5 +38,5 @@
             <!-- Output -->
             <odometry_frame>odom</odometry_frame>
-            <robot_base_frame>base</robot_base_frame>
+            <robot_base_frame>base_link</robot_base_frame><!-- was base -->
             <publish_odom>true</publish_odom>
             <publish_odom_tf>true</publish_odom_tf>
@@ -43,23 +45,21 @@
     </gazebo>
         <!-- GAZEBO JOINT STATE PUBLISHER -->
+        <!-- THIS IS NOT NEEDED ONCE HIGH LEVEL CONTROL IS ESTABLISHED -->
     <gazebo>
         <plugin name="gazebo_ros_joint_state_publisher" filename="libgazebo_ros_joint_state_publisher.so">
             <robotNamespace>/go1_gazebo</robotNamespace>
+            <update_rate>20</update_rate>
             <joint_name>FR_hip_joint</joint_name>
             <joint_name>FR_thigh_joint</joint_name>
             <joint_name>FR_calf_joint</joint_name>
-            <joint_name>FR_foot_joint</joint_name>
             <joint_name>FL_hip_joint</joint_name>
             <joint_name>FL_thigh_joint</joint_name>
             <joint_name>FL_calf_joint</joint_name>
-            <joint_name>FL_foot_joint</joint_name>
             <joint_name>RR_hip_joint</joint_name>
             <joint_name>RR_thigh_joint</joint_name>
             <joint_name>RR_calf_joint</joint_name>
-            <joint_name>RR_foot_joint</joint_name>
             <joint_name>RL_hip_joint</joint_name>
             <joint_name>RL_thigh_joint</joint_name>
             <joint_name>RL_calf_joint</joint_name>
-            <joint_name>RL_foot_joint</joint_name>
         </plugin>
     </gazebo>
@@ -74,5 +74,6 @@
             </plot>
         </plugin>
-    </gazebo> -->
+    </gazebo>
+    -->
     <!-- THIS GIVES ME A FAULT SAYING THE FORCE PLGIN NEEDS A <link_name> -->
     <!--
@@ -103,4 +104,5 @@
         </sensor>
     </gazebo>
+    <!-- THIS HAS TO BE COMMENTED OUT BECAUSE THE PLUGINS DONT EXIST FOR THE NEW VERSION OF GAZEBO ANYMORE, ONCE THEY BECOME AVAILIABLE THIS CAN BE USED -->
     <!-- Depth camera -->
     <!-- <gazebo>
@@ -223,5 +225,5 @@
     </gazebo>-->
     <!-- Foot contacts. -->
-    <!-- THIS I COMMENT OUT JUST TO TRY BECAUSE NEED PLUGIN FROM UNITREE-->
+    <!-- THIS HAS TO BE COMMENTED OUT UNTIL THE PLUGINS FOR ROS2 ARE AVAILIABLE FROM UNITREE -->
     <!--
     <gazebo reference="FR_calf">
@@ -263,5 +265,5 @@
     -->
     <!-- Visualization of Foot contacts. -->
-    <!-- THIS I COMMENT OUT JUST TO TRY BECAUSE NEED PLUGIN FROM UNITREE-->
+    <!-- THIS HAS TO BE COMMENTED OUT UNTIL THE PLUGINS FOR ROS2 ARE AVAILIABLE FROM UNITREE -->
     <!--
     <gazebo reference="FR_foot">
@@ -294,5 +296,5 @@
     </gazebo>
     -->
-    <gazebo reference="base">
+    <gazebo reference="base_link"><!-- was "base" -->
         <material>Gazebo/Green</material>
         <turnGravityOff>false</turnGravityOff>

File: xacro/robot.xacro (robot description, xacro)
@@ -9,6 +9,6 @@
     <!-- <xacro:include filename="$(find unigo1)/xacro/stairs.xacro"/> -->
     <xacro:include filename="$(find unigo1)/xacro/gazebo.xacro"/>
-    <xacro:include filename="$(find unigo1)/xacro/depthCamera.xacro"/>
-    <xacro:include filename="$(find unigo1)/xacro/ultraSound.xacro"/>
+    <xacro:include filename="$(find unigo1)/xacro/depthCamera1.xacro"/>
+<!--    <xacro:include filename="$(find unigo1)/xacro/ultraSound.xacro"/>-->
     <!-- <xacro:include filename="$(find go1_gazebo)/launch/stairs.urdf.xacro"/> -->
     <!-- <xacro:stairs stairs="15" xpos="0" ypos="0" zpos="0" /> -->
@@ -21,8 +21,8 @@
             <origin rpy="0 0 0" xyz="0 0 0"/>
             <parent link="world"/>
-            <child link="base"/>
+            <child link="base_link"/><!-- was "base"-->
         </joint>
     </xacro:if>
-    <link name="base">
+    <link name="base_link"><!-- was "base", needs to be called base_link for Nav2, or remap Nav2 commands -->
         <visual>
             <origin rpy="0 0 0" xyz="0 0 0"/>
@@ -46,5 +46,5 @@
     <joint name="floating_base" type="fixed">
         <origin rpy="0 0 0" xyz="0 0 0.35"/><!-- z value set to 0.35 so robot floats in the air, should be set to 0 if controlling with legs-->
-        <parent link="base"/>
+        <parent link="base_link"/><!-- was "base"-->
         <child link="trunk"/>
     </joint>
@@ -78,5 +78,5 @@
         <!-- LEFT WHEEL -->
     <joint name="left_wheel_joint" type="continuous">
-        <parent link="base"/>
+        <parent link="base_link"/><!-- was "base"-->
         <child link="left_wheel"/>
         <origin xyz="0 0.175 0" rpy="-${pi/2} 0 0"/>
@@ -84,10 +84,10 @@
     </joint>
     <link name="left_wheel">
-        <!--<visual>
-            <geometry>
-                <cylinder length="0.04" radius="0.05" />
-            </geometry>
-            <material name="blue"/>
-        </visual>-->
+        <visual>
+            <geometry>
+                <cylinder length="0.04" radius="0.05" />
+            </geometry>
+            <material name="blue"/>
+        </visual>
         <collision>
             <geometry>
@@ -104,5 +104,5 @@
         <!-- RIGHT WHEEL -->
     <joint name="right_wheel_joint" type="continuous">
-        <parent link="base"/>
+        <parent link="base_link"/><!-- was "base"-->
         <child link="right_wheel"/>
         <origin xyz="0 -0.175 0" rpy="${pi/2} 0 0"/>
@@ -110,10 +110,10 @@
     </joint>
     <link name="right_wheel">
-        <!--<visual>
-            <geometry>
-                <cylinder length="0.04" radius="0.05" />
-            </geometry>
-            <material name="blue"/>
-        </visual>-->
+        <visual>
+            <geometry>
+                <cylinder length="0.04" radius="0.05" />
+            </geometry>
+            <material name="blue"/>
+        </visual>
         <collision>
             <geometry>
@@ -135,10 +135,10 @@
     </joint>
     <link name="front_ball">
-        <!--<visual>
-            <geometry>
-                <sphere radius="0.05" />
-            </geometry>
-            <material name="blue"/>
-        </visual>-->
+        <visual>
+            <geometry>
+                <sphere radius="0.05" />
+            </geometry>
+            <material name="blue"/>
+        </visual>
         <collision>
             <geometry>
@@ -165,10 +165,10 @@
     </joint>
     <link name="back_ball">
-        <!--<visual>
-            <geometry>
-                <sphere radius="0.05" />
-            </geometry>
-            <material name="blue"/>
-        </visual>-->
+        <visual>
+            <geometry>
+                <sphere radius="0.05" />
+            </geometry>
+            <material name="blue"/>
+        </visual>
         <collision>
             <geometry>
@@ -221,4 +221,6 @@
         <origin rpy="${PI} 0 0" xyz="0.2785 0.0125 0.0167"/>
     </xacro:depthCamera>
+<!-- COMMENTED OUT TO TRY AND UPDATE REFRESH RATE, ALSO ONLY USING DEPTHCAMERA1 AND COMMENTING OUT ULTRASOUND AND -->
+<!--
     <xacro:depthCamera camID="2" name="chin">
         <origin rpy="${PI} ${PI/2} 0" xyz="0.2522 0.0125 -0.0436"/>
@@ -256,3 +258,4 @@
         <origin rpy="0 0 0" xyz="0.2747 0.0 -0.0088"/>
     </xacro:ultraSound>
+-->
 </robot>
